File: PowerConditioner.kicad_sch (KiCad schematic)
At the start: 10 parts, among them J2 YK9010223000G, J8 YK9010223000G, K1 2-1904025-3, K2 2-1904025-3, K3 2-1904025-3, U3 IPB017N10N5LFATMA1, U5 IPB017N10N5LFATMA1

Commit message: layout done
Parts:
- removed J2, J8: YK9010223000G, YK9010223000G, symbol YK9010223000G:YK9010223000G
- added J9: YK9010323000G, YK9010323000G:YK9010323000G, symbol YK9010323000G:YK9010323000G
- H1, H2: footprint (none) -> MountingHole:MountingHole_8.4mm_M8_Pad_Via
- K1: value 2-1904025-3 -> BATT-EDLC
- K2: value 2-1904025-3 -> SERIAL-PARALLEL
- K3: value 2-1904025-3 -> OUTPUT
- R1: footprint (none) -> Resistor_THT:R_Axial_DIN0207_L6.3mm_D2.5mm_P2.54mm_Vertical
- U3, U5: footprint PG-TO 263-7_INF -> IPB017N10N5LFATMA1:PG-TO 263-7_INF
Connections:
- net GND: now also J9.3, J9.4
- net NBM_VLO: now also J9.1, J9.2
- net at K3.30: now also J9.5, J9.6
Other:
- note added: "1,2:BYPASS OUT 3,4:GND 5,6:NBM HI"
- note removed: "Terminal For Inverter"

Commit message: Order to JLCPCB
Parts:
- K1, K2, K3: footprint 2-1904025-3:RELAY_2-1904025-3 -> A3K1CSP12VDC1.6D:A3K1CSP12VDC16D; symbol PC7150:2-1904025-3 -> A3K1CSP12VDC1.6D:A3K1CSP12VDC1.6D; Height (none) -> 24.5; Manufacturer_Name (none) -> CIT Relay & Switch; Manufacturer_Part_Number (none) -> A3K1CSP12VDC1.6D
Connections:
- net BATT+: now also K1.A87 (NC_1), K1.A88 (NC_2), K1.A89 (NC_3), K2.88 (NO_2), K2.89 (NO_3); no longer K1.87A
- net EDLC-: now also K2.31 (COM_2), K2.32 (COM_3)
- net GND: now also K2.A87 (NC_1), K2.A88 (NC_2), K2.A89 (NC_3); no longer K2.87A
- net NBM_VHI: now also K3.A87 (NC_1), K3.A88 (NC_2), K3.A89 (NC_3); no longer K3.87A
- net at H1.1, K1.30 (COM_1): now also K1.31 (COM_2), K1.32 (COM_3)
- net at J9.5, J9.6, K3.30 (COM_1): now also K3.31 (COM_2), K3.32 (COM_3)
- net at K1.87 (NO_1), U3.4 (DRAIN): now also K1.88 (NO_2), K1.89 (NO_3)
- no-connect marks 1 -> 3
Other:
- moved on the sheet: J9
